Commit message: Moved cell description files to aimen package.

File: mashes_workcell/urdf/wt03_head.xacro (robot description, xacro)
@@ -3,5 +3,5 @@
   <property name="pi" value="3.141592654" />
   <xacro:property name="tcp_frame">
-    <origin xyz="0.216 -0.022 0.474" rpy="${pi} -1.047197555 ${pi}" />
+    <origin xyz="0.2462 -0.0203 0.4320" rpy="${pi} -1.047197555 ${pi}" />
   </xacro:property>
   <!-- Head -->
@@ -9,5 +9,5 @@
     <visual>
       <geometry>
-        <mesh filename="package://etna_workcell/meshes/head_wt03/visual/head_wt03.stl" />
+        <mesh filename="package://mashes_workcell/meshes/head_wt03/visual/head_wt03.stl" />
       </geometry>
       <material name="dark_gray">
@@ -17,5 +17,5 @@
     <collision>
       <geometry>
-        <mesh filename="package://etna_workcell/meshes/head_wt03/collision/head_wt03.stl" />
+        <mesh filename="package://mashes_workcell/meshes/head_wt03/collision/head_wt03.stl" />
       </geometry>
       <material name="yellow">
