Commit message: Fixed some minor bugs.

File: mashes_workcell/urdf/workcell.urdf (robot description, URDF)
Before this commit: robot aimen_workcell, 25 links, 26 joints
Links:
- link base_link: geometry collision mesh filename=package://aimen_abb/meshes/irb4400/collision/base_link.stl; visual mesh filename=package://aimen_abb/meshes/irb4400/visual/base_link.stl
- link link_1: geometry collision mesh filename=package://aimen_abb/meshes/irb4400/collision/link_1.stl; visual mesh filename=package://aimen_abb/meshes/irb4400/visual/link_1.stl
- link link_2: geometry collision mesh filename=package://aimen_abb/meshes/irb4400/collision/link_2.stl; visual mesh filename=package://aimen_abb/meshes/irb4400/visual/link_2.stl
- link link_3: geometry collision mesh filename=package://aimen_abb/meshes/irb4400/collision/link_3.stl; visual mesh filename=package://aimen_abb/meshes/irb4400/visual/link_3.stl
- link link_4: geometry collision mesh filename=package://aimen_abb/meshes/irb4400/collision/link_4.stl; visual mesh filename=package://aimen_abb/meshes/irb4400/visual/link_4.stl
- link link_5: geometry collision mesh filename=package://aimen_abb/meshes/irb4400/collision/link_5.stl; visual mesh filename=package://aimen_abb/meshes/irb4400/visual/link_5.stl
- link link_6: geometry collision mesh filename=package://aimen_abb/meshes/irb4400/collision/link_6.stl; visual mesh filename=package://aimen_abb/meshes/irb4400/visual/link_6.stl
- link link_d1: geometry visual mesh filename=package://aimen_abb/meshes/irb4400/visual/link_d1.stl
- link link_d2: geometry visual mesh filename=package://aimen_abb/meshes/irb4400/visual/link_d2.stl
- link link_d3: geometry visual mesh filename=package://aimen_abb/meshes/irb4400/visual/link_d3.stl
- link link_d4: geometry visual mesh filename=package://aimen_abb/meshes/irb4400/visual/link_d4.stl
