Commit message: Refactored some joint names in workcell description.

File: mashes_workcell/urdf/workcell.xacro (robot description, xacro)
@@ -2,15 +2,16 @@
 <robot name="aimen_workcell" xmlns:xacro="http://ros.org/wiki/xacro">
   <property name="pi" value="3.141592654" />
+  <xacro:property name="tcp_frame">
+    <origin xyz="0.2462 -0.0203 0.4320" rpy="${pi} -1.047197555 ${pi}" />
+  </xacro:property>
   <xacro:property name="workobject_frame">
     <origin xyz="1.550 -0.185 0.930" rpy="0 0 0" />
   </xacro:property>
   <xacro:property name="camera_frame">
-    <!-- <origin xyz="0.0590 0.2170 0.3302" rpy="-1.161231 0.274247 -2.063781" /> -->
     <origin xyz="0.0715 0.2219 0.3248" rpy="-1.148206 0.311297 -2.151468" />
   </xacro:property>
-  <link name="world" />
-  <!-- Robot -->
-  <xacro:include filename="$(find aimen_workcell)/urdf/abb_robot.xacro"/>
-  <joint name="world-abb_robot" type="fixed">
+  <!-- Robot cell -->
+  <xacro:include filename="$(find aimen_workcell)/urdf/workcell.xacro"/>
+  <joint name="workcell" type="fixed">
     <parent link="world"/>
     <child link="base_link"/>
@@ -19,5 +20,5 @@
   <!-- Head -->
   <xacro:include filename="$(find mashes_workcell)/urdf/wt03_head.xacro"/>
-  <joint name="tool0-head0" type="fixed">
+  <joint name="head0" type="fixed">
     <parent link="tool0"/>
     <child link="head0"/>
@@ -25,17 +26,15 @@
     <axis xyz="0 0 1"/>
   </joint>
+  <!-- TCP -->
+  <link name="tcp0"/>
+  <joint name="tcp0" type="fixed">
+    <parent link="tool0"/>
+    <child link="tcp0"/>
+    <xacro:insert_block name="tcp_frame" />
+    <axis xyz="0 0 1"/>
+  </joint>
   <!-- Workobject -->
-  <link name="workobject">
-  <!--<visual>
-    <geometry>
-      <box size="0.5 0.5 0.25"/>
-    </geometry>
-    <origin xyz="0.25 0.25 0.125"/>
-    <material name="blue">
-      <color rgba="0.7 0.1 0.3 0.15"/>
-    </material>
-  </visual>-->
-  </link>
-  <joint name="world-workobject" type="fixed">
+  <link name="workobject" />
+  <joint name="workobject" type="fixed">
     <parent link="base_link" />
     <child link="workobject" />
@@ -44,25 +43,8 @@
   <!-- Camera -->
   <link name="camera0" />
-  <joint name="tool0-camera0" type="fixed">
+  <joint name="camera0" type="fixed">
     <parent link="tool0"/>
     <child link="camera0"/>
     <xacro:insert_block name="camera_frame" />
   </joint>
-  <!-- Cell walls -->
-  <link name="walls">
-  <visual>
-    <geometry>
-      <mesh filename="package://aimen_workcell/meshes/cell/cell.stl"/>
-    </geometry>
-    <origin xyz="0 0 0" />
-    <material name="white">
-      <color rgba="1 1 1 0.75"/>
-    </material>
-  </visual>
-  </link>
-  <joint name="world_to_walls" type="fixed">
-    <parent link="world" />
-    <child link="walls" />
-    <origin xyz="0 0 0" />
-  </joint>
 </robot>

File: mashes_workcell/urdf/wt03_head.xacro (robot description, xacro)
@@ -1,9 +1,4 @@
 <?xml version="1.0" ?>
 <robot name="wt03_head" xmlns:xacro="http://ros.org/wiki/xacro">
-  <property name="pi" value="3.141592654" />
-  <xacro:property name="tcp_frame">
-    <origin xyz="0.2462 -0.0203 0.4320" rpy="${pi} -1.047197555 ${pi}" />
-  </xacro:property>
-  <!-- Head -->
   <link name="head0">
     <visual>
@@ -24,11 +19,3 @@
     </collision>
   </link>
-  <!-- TCP -->
-  <link name="tcp0"/>
-  <joint name="tool0-tcp0" type="fixed">
-    <parent link="tool0"/>
-    <child link="tcp0"/>
-    <xacro:insert_block name="tcp_frame" />
-    <axis xyz="0 0 1"/>
-  </joint>
 </robot>

Commit message: Updated some camera configuration files.

File: mashes_workcell/urdf/workcell.xacro (robot description, xacro)
@@ -6,5 +6,5 @@
   </xacro:property>
   <xacro:property name="workobject_frame">
-    <origin xyz="1.550 -0.185 0.930" rpy="0 0 0" />
+    <origin xyz="1.550 -0.178 0.9308" rpy="0 0 0" />
   </xacro:property>
   <xacro:property name="camera_frame">

Commit message: Fixed tachyon temperature issue.

File: mashes_workcell/urdf/workcell.xacro (robot description, xacro)
@@ -9,5 +9,5 @@
   </xacro:property>
   <xacro:property name="camera_frame">
-    <origin xyz="0.0715 0.2219 0.3248" rpy="-1.148206 0.311297 -2.151468" />
+    <origin xyz="0.1071 0.2057 0.3395" rpy="1.073493 -0.312395 0.957637" />
   </xacro:property>
   <!-- Robot cell -->
